File: trove8.kicad_sch (KiCad schematic)
At the start: 44 parts, among them J1 CONN_INPUTS, J2 CONN_OUTPUTS, J3 USB_C, J4 Micro_SD_Card, M1 Module-mcu-0.7, M2 Module-power12-0.2, M3 Module-vr-0.1, M4 Module-knock-0.1, M5 Module-power5-0.2, M6 Module-input-0.1, U1 LIS2DW12TR, U2 JDY-33, U3 LPS22HB, U4 TJA1051T-3

Commit message: Standalone version without hellen-one
Parts:
- removed BT1: BATTERY_CR2032, Battery:BatteryHolder_Keystone_1060_1x2032, symbol art-electro-power:BATTERY_CR2032
- removed C1: 100n, hellen-one-common:C0603, symbol hellen-one-common:Cap
- removed D5: 1N4148WS, hellen-one-common:SOD-323, symbol hellen-one-common:1N4148WS
- removed D8, D9: B5819W, hellen-one-common:SOD-123, symbol hellen-one-common:1N4148WS
- removed M1: Module-mcu-0.7, hellen-one-mcu-0.7:mcu, symbol hellen-mcu:Module-mcu-0.7
- removed M2: Module-power12-0.2, hellen-one-power12-0.2:power12, symbol hellen-power12:Module-power12-0.2
- removed M3: Module-vr-0.1, hellen-one-vr-0.1:vr, symbol hellen-vr:Module-vr-0.1
- removed M4: Module-knock-0.1, hellen-one-knock-0.1:knock, symbol hellen-knock 0.1:Module-knock-0.1
- removed M5: Module-power5-0.2, hellen-one-power5-0.2:power5, symbol hellen-power5:Module-power5-0.2
- removed M6: Module-input-0.1, hellen-one-input-0.1:input, symbol hellen-input:Module-input-0.1
- removed S1, S2: Button_SPST, hellen-one-common:SMD-2_2.9x3.9x1.7, symbol hellen-one-common:Button_SPST
- added C9: 100n, Capacitor_SMD:C_0402_1005Metric, symbol hellen-one-common:Cap
- added D9: 1N5819WS, Diode_SMD:D_SOD-123, symbol Device:D_Schottky_Small
- added F11: 120mA, Fuse:Fuse_1206_3216Metric, symbol Device:Polyfuse
- added NT1: NetTie_2, NetTie:NetTie-2_SMD_Pad0.5mm, symbol Device:NetTie_2
- added U5: MPX4/MPXH6400_MAP, kicad6-libraries:MPX-4_MAP, symbol MPX-4_MAP:MPX4/MPXH6400_MAP
- added U6: USBLC6-2SC6, Package_TO_SOT_SMD:SOT-23-6, symbol proteus-rescue:USBLC6-2SC6-Power_Protection
- H1, H2, H3, H4: symbol Mechanical:MountingHole -> Mechanical:MountingHole_Pad; LCSC (none) -> NA; now left out of the parts list
- J1: LCSC (none) -> DNP; now left out of the parts list
- J2: footprint Connector_Automotive:Delphi_Sicma_24_Black -> Connector_Automotive:Delphi_Sicma_24_Grey; LCSC (none) -> DNP; now left out of the parts list
- U1: LCSC C189624 -> C50385411
- U4: renamed from U3; LCSC (none) -> C94049
- renumbered C4 to C1, C7 to C2, C5 to C3, C6 to C4, C8 to C5, C9 to C6, C2 to C7, C3 to C8, D6 to D7, D7 to D8, F2 to F1, U4 to U3
Connections:
- net +12V_IN: now also D1.1 (K), D2.1 (K), D3.1 (K), D4.1 (K)
- net +12V_RAW: no longer D1.1 (K), D2.1 (K), D3.1 (K), D4.1 (K)
- net +5V: now also D9.1 (K)
- net +5VA: now also C9.2, F11.1, U5.3 (VCC); no longer J1.C4
- net CAN1_RX: now also U3.4 (RXD); no longer U3.1 (TXD)
- net CAN1_TX: now also U3.1 (TXD); no longer U3.4 (RXD)
- net GND: now also H1.1, H2.1, H3.1, H4.1, C9.1, NT1.1, U5.2 (GND), U6.2 (GND); no longer J4.3 (CMD)
- net GNDA: now also NT1.2
- net IN_AC_CLUTCH: now also J1.C5; no longer J1.B7
- net IN_CAM_NEGATIVE: now also J1.A4; no longer J1.A3
- net IN_CAM_PRIMARY: now also J1.A3; no longer J1.A4
- net IN_CLT: now also J1.A7; no longer J1.B5
- net IN_CRANK_NEGATIVE: now also J1.A2; no longer J1.A1
- net IN_CRANK_PRIMARY: now also J1.A1; no longer J1.A2
- net IN_IAT: now also J1.A6; no longer J1.B6
- net IN_MAP: now also J1.A5; no longer J1.B4
- net IN_O2S: now also J1.B7; no longer J1.A5
- net IN_O2S2: now also J1.B6; no longer J1.A6
- net IN_PPS1: now also J1.B4; no longer J1.A8
- net IN_PPS2: now also J1.B5; no longer J1.A7
- net SD_CS: now also J4.2 (DAT3/CD); no longer J4.1 (DAT2)
- net SPI1_MOSI: now also J4.3 (CMD); no longer J4.2 (DAT3/CD)
- net USB_VBUS: now also D9.2 (A), U6.5 (VBUS)
- net +12V_KEY renamed +12V_PERM
- net OUT_LS5 renamed OUT_DH
- net OUT_LS6 renamed OUT_DL
- net USB+ renamed USB_D+
- net USB_D+: now also U6.3 (I/O2), U6.4 (I/O2)
- net USB- renamed USB_D-
- net USB_D-: now also U6.1 (I/O1), U6.6 (I/O1)
- new net: F11.2, J1.A8
- new net OUT: U5.1 (VOUT)
- no-connect marks 13 -> 15
Other:
- sheet LS6 renamed LS4
- added sheet Analog 1 (analog_input.kicad_sch)
- added sheet Analog 2 (analog_input.kicad_sch)
- added sheet Analog 3 Pullup (analog_input_pullup.kicad_sch)
- added sheet ETB (etb-9201.kicad_sch)
- added sheet Knock (knock.kicad_sch)
- added sheet MCU (mcu.kicad_sch)
- added sheet VR (vr.kicad_sch)
- added sheet VReg (VReg.kicad_sch)
- sheet LS4: file LS6.kicad_sch -> LS4.kicad_sch
- sheet LS4 ports: added none; removed IN5, IN6, OUT5, OUT6
- moved on the sheet: C1, C2, C3, C4, C5, C6, C7, C8, D1, D2, D3, D4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
