File: trove8.kicad_sch (KiCad schematic)
At the start: 37 parts, among them J1 CONN_INPUTS, J2 CONN_OUTPUTS, J3 USB_C, J4 Micro_SD_Card, U1 LIS2DW12TR, U2 JDY-33, U3 TJA1051T-3, U4 LPS22HB, U5 MPX4/MPXH6400_MAP, U6 USBLC6-2SC6

Commit message: Pre-cleanup
Parts:
- C1, C2, C3, C4, C5, C6, C7, C8, C9, D1, D2, D3, D4, D7: LCSC_ext (none) -> Basic
- D8, F1, F11, J3, J4: LCSC_ext (none) -> Extended
- D9: LCSC_ext 0 -> Basic
Connections:
- net IGN_1: now also J2.B1; no longer J2.A1
- net IGN_2: now also J2.B2; no longer J2.A2
- net IGN_3: now also J2.B3; no longer J2.A3
- net IGN_4: now also J2.B4; no longer J2.A4
- net IGN_5: now also J2.B5; no longer J2.A5
- net IGN_6: now also J2.B6; no longer J2.A6
- net IGN_7: now also J2.B7; no longer J2.A7
- net IGN_8: now also J2.B8; no longer J2.A8
- net INJ_1: now also J2.A1; no longer J2.B1
- net INJ_2: now also J2.A2; no longer J2.B2
- net INJ_3: now also J2.A3; no longer J2.B3
- net INJ_4: now also J2.A4; no longer J2.B4
- net INJ_5: now also J2.A5; no longer J2.B5
- net INJ_6: now also J2.A6; no longer J2.B6
- net INJ_7: now also J2.A7; no longer J2.B7
- net INJ_8: now also J2.A8; no longer J2.B8
- net IN_AC_CLUTCH: now also J1.B5; no longer J1.C5
- net IN_CAM_NEGATIVE: now also J1.A2; no longer J1.A4
- net IN_CAM_PRIMARY: now also J1.B2; no longer J1.A3
- net IN_CRANK_NEGATIVE: now also J1.A1; no longer J1.A2
- net IN_CRANK_PRIMARY: now also J1.B1; no longer J1.A1
- net IN_IAT: now also J1.B7; no longer J1.A6
- net IN_KNOCK: now also J1.C5; no longer J1.B1
- net IN_O2S: now also J1.A6; no longer J1.B7
- net IN_PPS1: now also J1.A4; no longer J1.B4
- net IN_PPS2: now also J1.B4; no longer J1.B5
- net IN_TPS_1: now also J1.A3; no longer J1.B2
- net IN_KNOCK2: now reaches J1.C4
Other:
- added sheet Knock1 (knock.kicad_sch)
- moved on the sheet: F1, J2A, J2B, NT1
