File: IGN8.kicad_sch (KiCad schematic)
At the start: 27 parts, among them U7 SN74LVC4245APWR

Commit message: Pre-cleanup
Parts:
- C10, C11: LCSC_ext (none) -> Basic
- F2, F3, F4, F5, F6, F7, F8, F9: LCSC_ext (none) -> Extended
