File: VReg.kicad_sch (KiCad schematic)
At the start: 35 parts, among them U14 LMR14020, U15 TLS115, U16 AMS1117-3.3, U25 MIC5205-3.3YM5

Commit message: Pre-cleanup
Parts:
- C12, C13, C14, C15, C17, C25, C26, C59, C78: LCSC_ext (none) -> Basic
- C16, C18, C19, C20, C21, C22, C24, D11, D12, D16, D17: LCSC_ext 0 -> Basic
- C23: footprint Capacitor_SMD:C_0402_1005Metric -> Capacitor_SMD:C_0603_1608Metric; LCSC C13533 -> C1664; LCSC_ext 0 -> Basic
- D10, L1, L2: LCSC_ext 1 -> Extended
- F10: LCSC_ext (none) -> Extended
