File: analog_input_pullup.kicad_sch (KiCad schematic)
At the start: 21 parts, among them U28 SRV05-4, U29 MCP6004

Commit message: Pre-cleanup
Parts:
- C72, C73, C74, C75, C76, C77: LCSC_ext 0 -> Basic
