File: mcu.kicad_sch (KiCad schematic)
At the start: 48 parts, among them J5 Conn_02x05_Odd_Even, J6 Conn_01x06, U26 STM32F427VGTx, Y1 20MHz, Y2 32.768 kHz

Commit message: Pre-cleanup
Parts:
- added U30: STM32F765VGTx, Package_QFP:LQFP-100_14x14mm_P0.5mm, symbol MCU_ST_STM32F7:STM32F765VGTx
- BOOT0: LCSC_ext 1 -> Basic
- C46, C47, C48, C49, C50, C51, C52, C53, C54, C55, C56, C57, C58, C60, C61, C62, C63, C64, C65, C66, D15, FB1, nRESET1: LCSC_ext 0 -> Basic
- C67, C68: value 12p -> 15p; LCSC C1547 -> C1548; LCSC_ext 0 -> Basic
- D13, D14, D5, D6: LCSC_ext (none) -> Basic
- U26: LCSC_ext (none) -> Extended
- Y2: footprint Crystal:Crystal_SMD_2012-2Pin_2.0x1.2mm -> Crystal:Crystal_SMD_3215-2Pin_3.2x1.5mm; LCSC C99009 -> C32346
Connections:
- new net: U30.10 (VSS), U30.26 (VSS), U30.49 (VSS), U30.74 (VSS), U30.99 (VSS)
