File: trove8.kicad_pcb (KiCad board)
At the start: 4 copper layers, 97 x 115 mm, 260 parts, among them J1 CONN_INPUTS, J2 CONN_OUTPUTS, J3 USB_C, J4 Micro_SD_Card, J6 Conn_01x06, U1 LIS2DW12TR, U10 VNLD5160TR-E, U11 VNLD5160TR-E, U12 VNLD5160TR-E, U13 VNLD5160TR-E, U14 LMR14020, U15 TLS115, U16 AMS1117-3.3, U17 SRV05-4, U18 MCP6004, U19 LMV321, U20 LMV321, U21 SRV05-4, U22 MCP6004, U23 MAX9924, U24 MAX9924, U25 MIC5205-3.3YM5, U26 STM32F427VGTx, U27 TLE9201SG, U28 SRV05-4, U29 MCP6004, U3 TJA1051T-3, U4 LPS22HB, U6 USBLC6-2SC6, U7 SN74LVC4245APWR, U8 VNLD5160TR-E, U9 VNLD5160TR-E, Y1 20MHz, Y2 32.768 kHz

Commit message: Pre-cleanup
Parts:
- added C79: 10n, Capacitor_SMD:C_0402_1005Metric, F.Cu at (133.0, 62.7)
- added C80: 3.3n, Capacitor_SMD:C_0603_1608Metric, F.Cu at (135.3, 57.7)
- added C81: 680p, Capacitor_SMD:C_0402_1005Metric, F.Cu at (136.1, 66.4)
- added C82: 330p, Capacitor_SMD:C_0603_1608Metric, F.Cu at (133.0, 69.5)
- added C83: 47p, Capacitor_SMD:C_0402_1005Metric, F.Cu at (136.1, 67.4)
- added R112: 33k, Resistor_SMD:R_0402_1005Metric, F.Cu at (133.0, 60.7)
- added R113: 33k, Resistor_SMD:R_0402_1005Metric, F.Cu at (134.2, 64.4)
- added R114: 100k, Resistor_SMD:R_0402_1005Metric, F.Cu at (136.0, 59.2)
- added R115: 470k, Resistor_SMD:R_0402_1005Metric, F.Cu at (136.1, 64.4)
- added R116: 12k, Resistor_SMD:R_0402_1005Metric, F.Cu at (136.1, 65.4)
- added R117: 100k, Resistor_SMD:R_0402_1005Metric, F.Cu at (134.2, 65.4)
- added R118: 33k, Resistor_SMD:R_0402_1005Metric, F.Cu at (134.2, 66.4)
- added U31: LMV321, Package_TO_SOT_SMD:SOT-23-5, F.Cu at (135.3, 61.8)
- added U32: LMV321, Package_TO_SOT_SMD:SOT-23-5, F.Cu at (135.5, 70.0)
- C23, C35: footprint Capacitor_SMD:C_0402_1005Metric -> Capacitor_SMD:C_0603_1608Metric
- C33: footprint Capacitor_SMD:C_0805_2012Metric -> Capacitor_SMD:C_0603_1608Metric
- C67, C68: value 12p -> 15p
- Y2: footprint Crystal:Crystal_SMD_2012-2Pin_2.0x1.2mm -> Crystal:Crystal_SMD_3215-2Pin_3.2x1.5mm
- moved U20 7.29 mm to (140.5, 70.0)
- moved U19 6.98 mm to (140.1, 61.8)
- moved C32 6.98 mm to (137.7, 62.7)
- moved R50 6.98 mm to (137.7, 60.7)
- moved C33 6.98 mm to (140.0, 57.7)
- moved C34 6.98 mm to (140.8, 66.4)
- moved C36 6.98 mm to (140.8, 67.4)
- moved R51 6.98 mm to (138.9, 64.4)
- moved R52 6.98 mm to (140.8, 59.2)
- moved R53 6.98 mm to (140.8, 64.4)
- moved R54 6.98 mm to (140.8, 65.4)
- moved R55 6.98 mm to (138.9, 65.4)
- moved R56 6.98 mm to (138.9, 66.4)
- moved BOOT0 6.33 mm to (156.3, 107.7)
- moved C63 6.33 mm to (155.2, 104.1)
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Connections:
- J1 pad A1: /IN_CRANK_PRIMARY -> /IN_CRANK_NEGATIVE
- J1 pad A2: /IN_CRANK_NEGATIVE -> /IN_CAM_NEGATIVE
- J1 pad A3: /IN_CAM_PRIMARY -> /IN_TPS_1
- J1 pad A4: /IN_CAM_NEGATIVE -> /IN_PPS1
- J1 pad A6: /IN_IAT -> /IN_O2S
- J1 pad B1: /IN_KNOCK -> /IN_CRANK_PRIMARY
- J1 pad B2: /IN_TPS_1 -> /IN_CAM_PRIMARY
- J1 pad B4: /IN_PPS1 -> /IN_PPS2
- J1 pad B5: /IN_PPS2 -> /IN_AC_CLUTCH
- J1 pad B7: /IN_O2S -> /IN_IAT
- J1 pad C4: unconnected-(J1-PadC4) -> /IN_KNOCK2
- J1 pad C5: /IN_AC_CLUTCH -> /IN_KNOCK
- J2 pad A1: /IGN_1 -> /INJ_1
- J2 pad A2: /IGN_2 -> /INJ_2
- J2 pad A3: /IGN_3 -> /INJ_3
- J2 pad A4: /IGN_4 -> /INJ_4
- J2 pad A5: /IGN_5 -> /INJ_5
- J2 pad A6: /IGN_6 -> /INJ_6
- J2 pad A7: /IGN_7 -> /INJ_7
- J2 pad A8: /IGN_8 -> /INJ_8
- J2 pad B1: /INJ_1 -> /IGN_1
- J2 pad B2: /INJ_2 -> /IGN_2
- J2 pad B3: /INJ_3 -> /IGN_3
- J2 pad B4: /INJ_4 -> /IGN_4
- J2 pad B5: /INJ_5 -> /IGN_5
- J2 pad B6: /INJ_6 -> /IGN_6
- J2 pad B7: /INJ_7 -> /IGN_7
- J2 pad B8: /INJ_8 -> /IGN_8
Routing:
- net GND: track 244.5 -> 204.6 mm, vias 124 -> 142
- net /IN_KNOCK2: track 0.00 -> 26.5 mm
- net +3.3V: track 423.6 -> 443.9 mm, vias 27 -> 29
- net /IN_TPS_1: track 34.6 -> 18.6 mm
- net /IN_O2S: track 29.2 -> 19.0 mm
- net /IN_PPS1: track 27.3 -> 17.8 mm, vias 1 -> 0
- net /IN_AC_CLUTCH: track 33.6 -> 25.1 mm, vias 1 -> 0
- net +5VA: track 145.9 -> 137.9 mm, vias 12 -> 11
- net /IN_TPS_2: track 30.6 -> 23.0 mm
- net /MCU_IN_KNOCK: track 25.5 -> 32.6 mm
- net /MCU_VREF: track 38.6 -> 45.1 mm
- net /MCU_IN_CLT: track 32.7 -> 39.1 mm
- net /MCU_IN_VIGN: track 36.1 -> 42.5 mm
- net /MCU_IN_IAT: track 31.2 -> 37.6 mm
- net /MCU_IN_PPS1: track 21.4 -> 27.8 mm
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