File: vr.kicad_sch (KiCad schematic)
At the start: 23 parts, among them U23 MAX9924, U24 MAX9924

Commit message: Pre-cleanup
Parts:
- C42, C43, C44, C45: LCSC_ext 0 -> Basic
Other:
- moved on the sheet: C45, JP1, R71, R72, R78, R83, R84
